File: hardware/Helios_Kicad/DAC.sch (KiCad schematic (older format))
At the start: 4 parts, among them U5 DAC084S085C

Commit message: redone pcb, driver and firmware working-ish
Parts:
- C11: renamed from C10; footprint Capacitors_SMD:C_0805 -> Capacitors_SMD:C_0603
- renumbered C9 to C10, C11 to C12
Connections:
- net G: now also U5.4 (Voutc); no longer U5.2 (Vouta)
- net Intensity: now also U5.2 (Vouta); no longer U5.4 (Voutc)
Changed lines of the file:
@@
 LIBS:valves
 LIBS:Personal library
+LIBS:Helios-cache
 EELAYER 25 0
 EELAYER END
@@
 Text HLabel 4550 4650 0    60   Output ~ 0
 R
-Text HLabel 4550 4350 0    60   Output ~ 0
+Text HLabel 4550 4550 0    60   Output ~ 0
 G
 Text HLabel 4550 4450 0    60   Output ~ 0
 B
 $Comp
-L C C9
+L C C10
 U 1 1 56B32431
 P 4600 3600
-F 0 "C9" H 4625 3700 50  0000 L CNN
+F 0 "C10" H 4625 3700 50  0000 L CNN
 F 1 "100nF" H 4625 3500 50  0000 L CNN
 F 2 "Capacitors_SMD:C_0402" H 4638 3450 50  0001 C CNN
@@
 Connection ~ 4600 4250
 $Comp
-L GND #PWR13
+L GND #PWR015
 U 1 1 56B430BD
 P 4600 3250
-F 0 "#PWR13" H 4600 3000 50  0001 C CNN
+F 0 "#PWR015" H 4600 3000 50  0001 C CNN
 F 1 "GND" H 4600 3100 50  0000 C CNN
 F 2 "" H 4600 3250 50  0000 C CNN
@@
 Wire Wire Line
 	4600 3250 4600 3450
-Text HLabel 4550 4550 0    60   Output ~ 0
+Text HLabel 4550 4350 0    60   Output ~ 0
 Intensity
 Wire Wire Line
 	4550 4650 4650 4650
 $Comp
-L C C10
+L C C11
 U 1 1 573A519D
 P 4900 3600
-F 0 "C10" H 4925 3700 50  0000 L CNN
+F 0 "C11" H 4925 3700 50  0000 L CNN
 F 1 "4.7uF" H 4925 3500 50  0000 L CNN
-F 2 "Capacitors_SMD:C_0805" H 4938 3450 50  0001 C CNN
+F 2 "Capacitors_SMD:C_0603" H 4938 3450 50  0001 C CNN
 F 3 "" H 4900 3600 50  0000 C CNN
 	1    4900 3600
@@
 Connection ~ 4600 3300
 $Comp
-L C C11
+L C C12
 U 1 1 57580D1C
 P 6450 4750
-F 0 "C11" H 6475 4850 50  0000 L CNN
+F 0 "C12" H 6475 4850 50  0000 L CNN
 F 1 "13pF" H 6475 4650 50  0000 L CNN
 F 2 "Capacitors_SMD:C_0402" H 6488 4600 50  0001 C CNN
@@
 $EndComp
 $Comp
-L GND #PWR15
+L GND #PWR016
 U 1 1 57580DA3
 P 6450 4950
-F 0 "#PWR15" H 6450 4700 50  0001 C CNN
+F 0 "#PWR016" H 6450 4700 50  0001 C CNN
 F 1 "GND" H 6450 4800 50  0000 C CNN
 F 2 "" H 6450 4950 50  0000 C CNN
@@
 Connection ~ 6450 4550
 $Comp
-L GND #PWR14
+L GND #PWR017
 U 1 1 575A7248
 P 5900 4650
-F 0 "#PWR14" H 5900 4400 50  0001 C CNN
+F 0 "#PWR017" H 5900 4400 50  0001 C CNN
 F 1 "GND" H 5900 4500 50  0000 C CNN
 F 2 "" H 5900 4650 50  0000 C CNN

Commit message: rev 1.1 pcb final
Parts:
- C11: footprint Capacitors_SMD:C_0603 -> Capacitors_SMD:c_elec_4x5.3
Changed lines of the file:
@@
 Connection ~ 4600 4250
 $Comp
-L GND #PWR015
+L GND #PWR13
 U 1 1 56B430BD
 P 4600 3250
-F 0 "#PWR015" H 4600 3000 50  0001 C CNN
+F 0 "#PWR13" H 4600 3000 50  0001 C CNN
 F 1 "GND" H 4600 3100 50  0000 C CNN
 F 2 "" H 4600 3250 50  0000 C CNN
@@
 F 0 "C11" H 4925 3700 50  0000 L CNN
 F 1 "4.7uF" H 4925 3500 50  0000 L CNN
-F 2 "Capacitors_SMD:C_0603" H 4938 3450 50  0001 C CNN
+F 2 "Capacitors_SMD:c_elec_4x5.3" H 4938 3450 50  0001 C CNN
 F 3 "" H 4900 3600 50  0000 C CNN
 	1    4900 3600
@@
 $EndComp
 $Comp
-L GND #PWR016
+L GND #PWR15
 U 1 1 57580DA3
 P 6450 4950
-F 0 "#PWR016" H 6450 4700 50  0001 C CNN
+F 0 "#PWR15" H 6450 4700 50  0001 C CNN
 F 1 "GND" H 6450 4800 50  0000 C CNN
 F 2 "" H 6450 4950 50  0000 C CNN
@@
 Connection ~ 6450 4550
 $Comp
-L GND #PWR017
+L GND #PWR14
 U 1 1 575A7248
 P 5900 4650
-F 0 "#PWR017" H 5900 4400 50  0001 C CNN
+F 0 "#PWR14" H 5900 4400 50  0001 C CNN
 F 1 "GND" H 5900 4500 50  0000 C CNN
 F 2 "" H 5900 4650 50  0000 C CNN
