File: hardware/Helios_Kicad/Microcontroller.sch (KiCad schematic (older format))
At the start: 24 parts, among them P3 CONN_01X03, U9 ATSAM4S, Y1 16MHz 18pF

Commit message: redone pcb, driver and firmware working-ish
Parts:
- removed P3: CONN_01X03, Pin_Headers:Pin_Header_Straight_1x03, symbol CONN_01X03
- added P3: CONN_01X02, Connect:PINHEAD1-2, symbol CONN_01X02
- C23: renamed from C22; footprint Capacitors_SMD:C_0805 -> Capacitors_SMD:C_0603
- C24: renamed from C23; footprint Capacitors_SMD:C_0805 -> Capacitors_SMD:C_0603
- C30: renamed from C29; footprint Capacitors_SMD:C_0805 -> Capacitors_SMD:C_0603
- renumbered C18 to C19, C19 to C20, C20 to C21, C21 to C22, C24 to C25, C25 to C26, C26 to C27, C27 to C28, C28 to C29, C30 to C31, C31 to C32, L2 to L3, R42 to R45, R40 to R46, R41 to R47, R43 to R48
Connections:
- net 3.3V: now also P3.2 (P2)
- net ERASE: now also P3.1 (P1)
- no-connect marks 37 -> 36
Changed lines of the file:
@@
 LIBS:valves
 LIBS:Personal library
+LIBS:Helios-cache
 EELAYER 25 0
 EELAYER END
@@
 3.3V
 $Comp
-L C C20
+L C C21
 U 1 1 56B26047
 P 2400 1600
-F 0 "C20" H 2425 1700 50  0000 L CNN
+F 0 "C21" H 2425 1700 50  0000 L CNN
 F 1 "100nF" H 2425 1500 50  0000 L CNN
 F 2 "Capacitors_SMD:C_0402" H 2438 1450 50  0001 C CNN
@@
 $EndComp
 $Comp
-L GND #PWR31
+L GND #PWR033
 U 1 1 56B2611E
 P 2400 2100
-F 0 "#PWR31" H 2400 1850 50  0001 C CNN
+F 0 "#PWR033" H 2400 1850 50  0001 C CNN
 F 1 "GND" H 2400 1950 50  0000 C CNN
 F 2 "" H 2400 2100 50  0000 C CNN
@@
 $EndComp
 $Comp
-L GND #PWR32
+L GND #PWR034
 U 1 1 56B261DD
 P 2500 3400
-F 0 "#PWR32" H 2500 3150 50  0001 C CNN
+F 0 "#PWR034" H 2500 3150 50  0001 C CNN
 F 1 "GND" H 2500 3250 50  0000 C CNN
 F 2 "" H 2500 3400 50  0000 C CNN
@@
 $EndComp
 $Comp
-L C C23
+L C C24
 U 1 1 56B263C7
 P 2700 4600
-F 0 "C23" H 2725 4700 50  0000 L CNN
+F 0 "C24" H 2725 4700 50  0000 L CNN
 F 1 "4.7uF" H 2725 4500 50  0000 L CNN
-F 2 "Capacitors_SMD:C_0805" H 2738 4450 50  0001 C CNN
+F 2 "Capacitors_SMD:C_0603" H 2738 4450 50  0001 C CNN
 F 3 "" H 2700 4600 50  0000 C CNN
 	1    2700 4600
@@
 $EndComp
 $Comp
-L GND #PWR33
+L GND #PWR035
 U 1 1 56B264E0
 P 3300 5150
-F 0 "#PWR33" H 3300 4900 50  0001 C CNN
+F 0 "#PWR035" H 3300 4900 50  0001 C CNN
 F 1 "GND" H 3300 5000 50  0000 C CNN
 F 2 "" H 3300 5150 50  0000 C CNN
@@
 3.3V
 $Comp
-L C C28
+L C C29
 U 1 1 56B28036
 P 3600 7050
-F 0 "C28" H 3625 7150 50  0000 L CNN
+F 0 "C29" H 3625 7150 50  0000 L CNN
 F 1 "13pF" H 3625 6950 50  0000 L CNN
 F 2 "Capacitors_SMD:C_0402" H 3638 6900 50  0001 C CNN
@@
 $EndComp
 $Comp
-L C C30
+L C C31
 U 1 1 56B2808A
 P 4400 7050
-F 0 "C30" H 4425 7150 50  0000 L CNN
+F 0 "C31" H 4425 7150 50  0000 L CNN
 F 1 "13pF" H 4425 6950 50  0000 L CNN
 F 2 "Capacitors_SMD:C_0402" H 4438 6900 50  0001 C CNN
@@
 $EndComp
 $Comp
-L GND #PWR34
+L GND #PWR036
 U 1 1 56B28207
 P 3600 7400
-F 0 "#PWR34" H 3600 7150 50  0001 C CNN
+F 0 "#PWR036" H 3600 7150 50  0001 C CNN
 F 1 "GND" H 3600 7250 50  0000 C CNN
 F 2 "" H 3600 7400 50  0000 C CNN
@@
 $EndComp
 $Comp
-L GND #PWR35
+L GND #PWR037
 U 1 1 56B282D6
 P 4400 7400
-F 0 "#PWR35" H 4400 7150 50  0001 C CNN
+F 0 "#PWR037" H 4400 7150 50  0001 C CNN
 F 1 "GND" H 4400 7250 50  0000 C CNN
 F 2 "" H 4400 7400 50  0000 C CNN
@@
 $EndComp
 $Comp
-L GND #PWR36
+L GND #PWR038
 U 1 1 56BC9489
 P 5200 7450
-F 0 "#PWR36" H 5200 7200 50  0001 C CNN
+F 0 "#PWR038" H 5200 7200 50  0001 C CNN
 F 1 "GND" H 5200 7300 50  0000 C CNN
 F 2 "" H 5200 7450 50  0000 C CNN
@@
 $EndComp
 $Comp
-L GND #PWR37
+L GND #PWR039
 U 1 1 56BC94D0
 P 5550 7450
-F 0 "#PWR37" H 5550 7200 50  0001 C CNN
+F 0 "#PWR039" H 5550 7200 50  0001 C CNN
 F 1 "GND" H 5550 7300 50  0000 C CNN
 F 2 "" H 5550 7450 50  0000 C CNN
@@
 $EndComp
 $Comp
-L R R41
+L R R47
 U 1 1 56BC9811
 P 5550 6850
-F 0 "R41" V 5630 6850 50  0000 C CNN
+F 0 "R47" V 5630 6850 50  0000 C CNN
 F 1 "1.65k" V 5550 6850 50  0000 C CNN
 F 2 "Resistors_SMD:R_0603" V 5480 6850 50  0001 C CNN
@@
 $EndComp
 $Comp
-L R R40
+L R R46
 U 1 1 56BC99C9
 P 5200 6850
-F 0 "R40" V 5280 6850 50  0000 C CNN
+F 0 "R46" V 5280 6850 50  0000 C CNN
 F 1 "1.65k" V 5200 6850 50  0000 C CNN
 F 2 "Resistors_SMD:R_0603" V 5130 6850 50  0001 C CNN
@@
 VDDIO
 $Comp
-L GND #PWR39
+L GND #PWR040
 U 1 1 56F0F05F
 P 6150 3400
-F 0 "#PWR39" H 6150 3150 50  0001 C CNN
+F 0 "#PWR040" H 6150 3150 50  0001 C CNN
 F 1 "GND" H 6150 3250 50  0000 C CNN
 F 2 "" H 6150 3400 50  0000 C CNN
@@
 VDDIO
 $Comp
-L GND #PWR43
+L GND #PWR041
 U 1 1 56F110A4
 P 8400 4500
-F 0 "#PWR43" H 8400 4250 50  0001 C CNN
+F 0 "#PWR041" H 8400 4250 50  0001 C CNN
 F 1 "GND" H 8400 4350 50  0000 C CNN
 F 2 "" H 8400 4500 50  0000 C CNN
@@
 NRST
 $Comp
-L GND #PWR42
+L GND #PWR042
 U 1 1 56F12B31
 P 8400 3100
-F 0 "#PWR42" H 8400 2850 50  0001 C CNN
+F 0 "#PWR042" H 8400 2850 50  0001 C CNN
 F 1 "GND" H 8400 2950 50  0000 C CNN
 F 2 "" H 8400 3100 50  0000 C CNN
@@
 VDDIN
 $Comp
-L GND #PWR40
+L GND #PWR043
 U 1 1 56F13C65
 P 6200 1900
-F 0 "#PWR40" H 6200 1650 50  0001 C CNN
+F 0 "#PWR043" H 6200 1650 50  0001 C CNN
 F 1 "GND" H 6200 1750 50  0000 C CNN
 F 2 "" H 6200 1900 50  0000 C CNN
@@
 Text Label 3500 1300 0    39   ~ 0
 VDDIO
-$Comp
-L CONN_01X03 P3
-U 1 1 573B1094
-P 1200 7250
-F 0 "P3" H 1200 7450 50  0000 C CNN
-F 1 "CONN_01X03" V 1300 7250 50  0000 C CNN
-F 2 "Pin_Headers:Pin_Header_Straight_1x03" H 1200 7250 50  0001 C CNN
-F 3 "" H 1200 7250 50  0000 C CNN
-	1    1200 7250
-	0    1    1    0
-$EndComp
-NoConn ~ 1300 7050
 NoConn ~ 6300 2000
 NoConn ~ 6300 2100
@@
 NoConn ~ 8300 3800
 $Comp
-L C C29
+L C C30
 U 1 1 573924C5
 P 3700 4600
-F 0 "C29" H 3725 4700 50  0000 L CNN
+F 0 "C30" H 3725 4700 50  0000 L CNN
 F 1 "4.7uF" H 3725 4500 50  0000 L CNN
-F 2 "Capacitors_SMD:C_0805" H 3738 4450 50  0001 C CNN
+F 2 "Capacitors_SMD:C_0603" H 3738 4450 50  0001 C CNN
 F 3 "" H 3700 4600 50  0000 C CNN
 	1    3700 4600
@@
 $EndComp
 $Comp
-L C C22
+L C C23
 U 1 1 573A58D9
 P 2500 3150
-F 0 "C22" H 2525 3250 50  0000 L CNN
+F 0 "C23" H 2525 3250 50  0000 L CNN
 F 1 "4.7uF" H 2525 3050 50  0000 L CNN
-F 2 "Capacitors_SMD:C_0805" H 2538 3000 50  0001 C CNN
+F 2 "Capacitors_SMD:C_0603" H 2538 3000 50  0001 C CNN
 F 3 "" H 2500 3150 50  0000 C CNN
 	1    2500 3150
@@
 NoConn ~ 8300 1900
 $Comp
-L C C24
+L C C25
 U 1 1 573BE091
 P 2800 1600
-F 0 "C24" H 2825 1700 50  0000 L CNN
+F 0 "C25" H 2825 1700 50  0000 L CNN
 F 1 "100nF" H 2825 1500 50  0000 L CNN
 F 2 "Capacitors_SMD:C_0402" H 2838 1450 50  0001 C CNN
@@
 $EndComp
 $Comp
-L C C26
+L C C27
 U 1 1 573BE0E9
 P 3150 1600
-F 0 "C26" H 3175 1700 50  0000 L CNN
+F 0 "C27" H 3175 1700 50  0000 L CNN
 F 1 "100nF" H 3175 1500 50  0000 L CNN
 F 2 "Capacitors_SMD:C_0402" H 3188 1450 50  0001 C CNN
@@
 $EndComp
 $Comp
-L C C25
+L C C26
 U 1 1 573BE1A6
 P 2900 3150
-F 0 "C25" H 2925 3250 50  0000 L CNN
+F 0 "C26" H 2925 3250 50  0000 L CNN
 F 1 "100nF" H 2925 3050 50  0000 L CNN
 F 2 "Capacitors_SMD:C_0402" H 2938 3000 50  0001 C CNN
@@
 $EndComp
 $Comp
-L C C27
+L C C28
 U 1 1 573BE20D
 P 3300 4600
-F 0 "C27" H 3325 4700 50  0000 L CNN
+F 0 "C28" H 3325 4700 50  0000 L CNN
 F 1 "100nF" H 3325 4500 50  0000 L CNN
 F 2 "Capacitors_SMD:C_0402" H 3338 4450 50  0001 C CNN
@@
 $EndComp
 $Comp
-L C C21
+L C C22
 U 1 1 573BE289
 P 2400 4600
-F 0 "C21" H 2425 4700 50  0000 L CNN
+F 0 "C22" H 2425 4700 50  0000 L CNN
 F 1 "100nF" H 2425 4500 50  0000 L CNN
 F 2 "Capacitors_SMD:C_0402" H 2438 4450 50  0001 C CNN
@@
 $EndComp
 $Comp
-L C C19
+L C C20
 U 1 1 573BE2F6
 P 2100 4600
-F 0 "C19" H 2125 4700 50  0000 L CNN
+F 0 "C20" H 2125 4700 50  0000 L CNN
 F 1 "100nF" H 2125 4500 50  0000 L CNN
 F 2 "Capacitors_SMD:C_0402" H 2138 4450 50  0001 C CNN
@@
 $EndComp
 $Comp
-L C C18
+L C C19
 U 1 1 573BE34A
 P 1800 4600
-F 0 "C18" H 1825 4700 50  0000 L CNN
+F 0 "C19" H 1825 4700 50  0000 L CNN
 F 1 "100nF" H 1825 4500 50  0000 L CNN
 F 2 "Capacitors_SMD:C_0402" H 1838 4450 50  0001 C CNN
@@
 $EndComp
 $Comp
-L GND #PWR41
+L GND #PWR044
 U 1 1 575A0181
 P 8300 2500
-F 0 "#PWR41" H 8300 2250 50  0001 C CNN
+F 0 "#PWR044" H 8300 2250 50  0001 C CNN
 F 1 "GND" H 8300 2350 50  0000 C CNN
 F 2 "" H 8300 2500 50  0000 C CNN
@@
 NoConn ~ 8400 2400
 $Comp
-L GND #PWR38
+L GND #PWR045
 U 1 1 575C07BB
 P 5750 2200
-F 0 "#PWR38" H 5750 1950 50  0001 C CNN
+F 0 "#PWR045" H 5750 1950 50  0001 C CNN
 F 1 "GND" H 5750 2050 50  0000 C CNN
 F 2 "" H 5750 2200 50  0000 C CNN
@@
 $EndComp
 $Comp
-L C C31
+L C C32
 U 1 1 575B717E
 P 5750 2050
-F 0 "C31" H 5775 2150 50  0000 L CNN
+F 0 "C32" H 5775 2150 50  0000 L CNN
 F 1 "13pF" H 5775 1950 50  0000 L CNN
 F 2 "Capacitors_SMD:C_0402" H 5788 1900 50  0001 C CNN
@@
 Text Label 5200 6450 0    39   ~ 0
 PA23
-Text HLabel 950  6950 0    60   Output ~ 0
-ERASE
 Wire Wire Line
 	5550 7000 5550 7050
 Wire Wire Line
 	5200 7000 5200 7050
-Connection ~ 1100 6950
-Wire Wire Line
-	1100 6950 950  6950
 Connection ~ 5750 1800
 Wire Wire Line
@@
 	6300 3100 6150 3100
 $Comp
-L R R42
+L R R45
 U 1 1 57603E8D
 P 5000 6850
-F 0 "R42" V 5080 6850 50  0000 C CNN
+F 0 "R45" V 5080 6850 50  0000 C CNN
 F 1 "1.65k" V 5000 6850 50  0000 C CNN
 F 2 "Resistors_SMD:R_0603" V 4930 6850 50  0001 C CNN
@@
 $EndComp
 $Comp
-L R R43
+L R R48
 U 1 1 57603EE8
 P 5750 6850
-F 0 "R43" V 5830 6850 50  0000 C CNN
+F 0 "R48" V 5830 6850 50  0000 C CNN
 F 1 "1.65k" V 5750 6850 50  0000 C CNN
 F 2 "Resistors_SMD:R_0603" V 5680 6850 50  0001 C CNN
@@
 Connection ~ 5550 6650
 $Comp
-L FILTER L2
+L FILTER L3
 U 1 1 5761B352
 P 3000 4300
-F 0 "L2" H 3000 4450 50  0000 C CNN
+F 0 "L3" H 3000 4450 50  0000 C CNN
 F 1 "FILTER" H 3000 4200 50  0000 C CNN
 F 2 "Resistors_SMD:R_0603" H 3000 4300 50  0001 C CNN
@@
 Wire Wire Line
 	3300 4400 3900 4400
+$Comp
+L CONN_01X02 P3
+U 1 1 5792C984
+P 1150 7250
+F 0 "P3" H 1150 7400 50  0000 C CNN
+F 1 "CONN_01X02" V 1250 7250 50  0000 C CNN
+F 2 "Connect:PINHEAD1-2" H 1150 7250 50  0001 C CNN
+F 3 "" H 1150 7250 50  0000 C CNN
+	1    1150 7250
+	0    -1   1    0
+$EndComp
 $EndSCHEMATC

Commit message: rev 1.1 pcb final
Parts:
- C23, C24, C30: footprint Capacitors_SMD:C_0603 -> Capacitors_SMD:c_elec_4x5.3
- renumbered P3 to ERASE1
Changed lines of the file:
@@
 $EndComp
 $Comp
-L GND #PWR033
+L GND #PWR31
 U 1 1 56B2611E
 P 2400 2100
-F 0 "#PWR033" H 2400 1850 50  0001 C CNN
+F 0 "#PWR31" H 2400 1850 50  0001 C CNN
 F 1 "GND" H 2400 1950 50  0000 C CNN
 F 2 "" H 2400 2100 50  0000 C CNN
@@
 $EndComp
 $Comp
-L GND #PWR034
+L GND #PWR32
 U 1 1 56B261DD
 P 2500 3400
-F 0 "#PWR034" H 2500 3150 50  0001 C CNN
+F 0 "#PWR32" H 2500 3150 50  0001 C CNN
 F 1 "GND" H 2500 3250 50  0000 C CNN
 F 2 "" H 2500 3400 50  0000 C CNN
@@
 F 0 "C24" H 2725 4700 50  0000 L CNN
 F 1 "4.7uF" H 2725 4500 50  0000 L CNN
-F 2 "Capacitors_SMD:C_0603" H 2738 4450 50  0001 C CNN
+F 2 "Capacitors_SMD:c_elec_4x5.3" H 2738 4450 50  0001 C CNN
 F 3 "" H 2700 4600 50  0000 C CNN
 	1    2700 4600
@@
 $EndComp
 $Comp
-L GND #PWR035
+L GND #PWR33
 U 1 1 56B264E0
 P 3300 5150
-F 0 "#PWR035" H 3300 4900 50  0001 C CNN
+F 0 "#PWR33" H 3300 4900 50  0001 C CNN
 F 1 "GND" H 3300 5000 50  0000 C CNN
 F 2 "" H 3300 5150 50  0000 C CNN
@@
 $EndComp
 $Comp
-L GND #PWR036
+L GND #PWR34
 U 1 1 56B28207
 P 3600 7400
-F 0 "#PWR036" H 3600 7150 50  0001 C CNN
+F 0 "#PWR34" H 3600 7150 50  0001 C CNN
 F 1 "GND" H 3600 7250 50  0000 C CNN
 F 2 "" H 3600 7400 50  0000 C CNN
@@
 $EndComp
 $Comp
-L GND #PWR037
+L GND #PWR35
 U 1 1 56B282D6
 P 4400 7400
-F 0 "#PWR037" H 4400 7150 50  0001 C CNN
+F 0 "#PWR35" H 4400 7150 50  0001 C CNN
 F 1 "GND" H 4400 7250 50  0000 C CNN
 F 2 "" H 4400 7400 50  0000 C CNN
@@
 $EndComp
 $Comp
-L GND #PWR038
+L GND #PWR36
 U 1 1 56BC9489
 P 5200 7450
-F 0 "#PWR038" H 5200 7200 50  0001 C CNN
+F 0 "#PWR36" H 5200 7200 50  0001 C CNN
 F 1 "GND" H 5200 7300 50  0000 C CNN
 F 2 "" H 5200 7450 50  0000 C CNN
@@
 $EndComp
 $Comp
-L GND #PWR039
+L GND #PWR37
 U 1 1 56BC94D0
 P 5550 7450
-F 0 "#PWR039" H 5550 7200 50  0001 C CNN
+F 0 "#PWR37" H 5550 7200 50  0001 C CNN
 F 1 "GND" H 5550 7300 50  0000 C CNN
 F 2 "" H 5550 7450 50  0000 C CNN
@@
 VDDIO
 $Comp
-L GND #PWR040
+L GND #PWR39
 U 1 1 56F0F05F
 P 6150 3400
-F 0 "#PWR040" H 6150 3150 50  0001 C CNN
+F 0 "#PWR39" H 6150 3150 50  0001 C CNN
 F 1 "GND" H 6150 3250 50  0000 C CNN
 F 2 "" H 6150 3400 50  0000 C CNN
@@
 VDDIO
 $Comp
-L GND #PWR041
+L GND #PWR43
 U 1 1 56F110A4
 P 8400 4500
-F 0 "#PWR041" H 8400 4250 50  0001 C CNN
+F 0 "#PWR43" H 8400 4250 50  0001 C CNN
 F 1 "GND" H 8400 4350 50  0000 C CNN
 F 2 "" H 8400 4500 50  0000 C CNN
@@
 NRST
 $Comp
-L GND #PWR042
+L GND #PWR42
 U 1 1 56F12B31
 P 8400 3100
-F 0 "#PWR042" H 8400 2850 50  0001 C CNN
+F 0 "#PWR42" H 8400 2850 50  0001 C CNN
 F 1 "GND" H 8400 2950 50  0000 C CNN
 F 2 "" H 8400 3100 50  0000 C CNN
@@
 VDDIN
 $Comp
-L GND #PWR043
+L GND #PWR40
 U 1 1 56F13C65
 P 6200 1900
-F 0 "#PWR043" H 6200 1650 50  0001 C CNN
+F 0 "#PWR40" H 6200 1650 50  0001 C CNN
 F 1 "GND" H 6200 1750 50  0000 C CNN
 F 2 "" H 6200 1900 50  0000 C CNN
@@
 F 0 "C30" H 3725 4700 50  0000 L CNN
 F 1 "4.7uF" H 3725 4500 50  0000 L CNN
-F 2 "Capacitors_SMD:C_0603" H 3738 4450 50  0001 C CNN
+F 2 "Capacitors_SMD:c_elec_4x5.3" H 3738 4450 50  0001 C CNN
 F 3 "" H 3700 4600 50  0000 C CNN
 	1    3700 4600
@@
 F 0 "C23" H 2525 3250 50  0000 L CNN
 F 1 "4.7uF" H 2525 3050 50  0000 L CNN
-F 2 "Capacitors_SMD:C_0603" H 2538 3000 50  0001 C CNN
+F 2 "Capacitors_SMD:c_elec_4x5.3" H 2538 3000 50  0001 C CNN
 F 3 "" H 2500 3150 50  0000 C CNN
 	1    2500 3150
@@
 $EndComp
 $Comp
-L GND #PWR044
+L GND #PWR41
 U 1 1 575A0181
 P 8300 2500
-F 0 "#PWR044" H 8300 2250 50  0001 C CNN
+F 0 "#PWR41" H 8300 2250 50  0001 C CNN
 F 1 "GND" H 8300 2350 50  0000 C CNN
 F 2 "" H 8300 2500 50  0000 C CNN
@@
 NoConn ~ 8400 2400
 $Comp
-L GND #PWR045
+L GND #PWR38
 U 1 1 575C07BB
 P 5750 2200
-F 0 "#PWR045" H 5750 1950 50  0001 C CNN
+F 0 "#PWR38" H 5750 1950 50  0001 C CNN
 F 1 "GND" H 5750 2050 50  0000 C CNN
 F 2 "" H 5750 2200 50  0000 C CNN
@@
 	3300 4400 3900 4400
 $Comp
-L CONN_01X02 P3
+L CONN_01X02 ERASE1
 U 1 1 5792C984
 P 1150 7250
-F 0 "P3" H 1150 7400 50  0000 C CNN
+F 0 "ERASE1" H 1150 7400 50  0000 C CNN
 F 1 "CONN_01X02" V 1250 7250 50  0000 C CNN
 F 2 "Connect:PINHEAD1-2" H 1150 7250 50  0001 C CNN
