File: hardware/Kicad_PCB_helios/Amplifiers.sch (KiCad schematic (older format))
At the start: 38 parts, among them U6 TL084_v, U7 LM358, U8 TL084_v

Commit message: pull
Parts:
- C13, C14, C15, C16, C17, C18: footprint Capacitors_SMD:C_0402 -> Capacitors_SMD:C_0603
Changed lines of the file:
@@
 EESchema Schematic File Version 2
+LIBS:Helios-rescue
 LIBS:power
 LIBS:device
@@
 2.5V
 $Comp
-L GND #PWR16
+L GND #PWR029
 U 1 1 56D62C05
 P 900 6950
-F 0 "#PWR16" H 900 6700 50  0001 C CNN
+F 0 "#PWR029" H 900 6700 50  0001 C CNN
 F 1 "GND" H 900 6800 50  0000 C CNN
 F 2 "" H 900 6950 50  0000 C CNN
@@
 $EndComp
 $Comp
-L GND #PWR22
+L GND #PWR030
 U 1 1 56D64930
 P 4600 7450
-F 0 "#PWR22" H 4600 7200 50  0001 C CNN
+F 0 "#PWR030" H 4600 7200 50  0001 C CNN
 F 1 "GND" H 4600 7300 50  0000 C CNN
 F 2 "" H 4600 7450 50  0000 C CNN
@@
 $EndComp
 $Comp
-L GND #PWR19
+L GND #PWR031
 U 1 1 56E9F32E
 P 2800 7400
-F 0 "#PWR19" H 2800 7150 50  0001 C CNN
+F 0 "#PWR031" H 2800 7150 50  0001 C CNN
 F 1 "GND" H 2800 7250 50  0000 C CNN
 F 2 "" H 2800 7400 50  0000 C CNN
@@
 +9V
 $Comp
-L GND #PWR26
+L GND #PWR032
 U 1 1 56EA45CC
 P 9450 5000
-F 0 "#PWR26" H 9450 4750 50  0001 C CNN
+F 0 "#PWR032" H 9450 4750 50  0001 C CNN
 F 1 "GND" H 9450 4850 50  0000 C CNN
 F 2 "" H 9450 5000 50  0000 C CNN
@@
 -9V
 $Comp
-L GND #PWR17
+L GND #PWR033
 U 1 1 56EA914F
 P 1350 2350
-F 0 "#PWR17" H 1350 2100 50  0001 C CNN
+F 0 "#PWR033" H 1350 2100 50  0001 C CNN
 F 1 "GND" H 1350 2200 50  0000 C CNN
 F 2 "" H 1350 2350 50  0000 C CNN
@@
 -9V
 $Comp
-L GND #PWR18
+L GND #PWR034
 U 1 1 56EAC37C
 P 1350 4200
-F 0 "#PWR18" H 1350 3950 50  0001 C CNN
+F 0 "#PWR034" H 1350 3950 50  0001 C CNN
 F 1 "GND" H 1350 4050 50  0000 C CNN
 F 2 "" H 1350 4200 50  0000 C CNN
@@
 -9V
 $Comp
-L GND #PWR20
+L GND #PWR035
 U 1 1 56EADE6C
 P 3650 4150
-F 0 "#PWR20" H 3650 3900 50  0001 C CNN
+F 0 "#PWR035" H 3650 3900 50  0001 C CNN
 F 1 "GND" H 3650 4000 50  0000 C CNN
 F 2 "" H 3650 4150 50  0000 C CNN
@@
 F 0 "C13" H 9460 1320 50  0000 L CNN
 F 1 "100nF" H 9460 1170 50  0000 L CNN
-F 2 "Capacitors_SMD:C_0402" H 9450 1250 50  0001 C CNN
+F 2 "Capacitors_SMD:C_0603" H 9450 1250 50  0001 C CNN
 F 3 "" H 9450 1250 50  0000 C CNN
 	1    9450 1250
@@
 +9V
 $Comp
-L GND #PWR23
+L GND #PWR036
 U 1 1 56ECCA82
 P 9450 1400
-F 0 "#PWR23" H 9450 1150 50  0001 C CNN
+F 0 "#PWR036" H 9450 1150 50  0001 C CNN
 F 1 "GND" H 9450 1250 50  0000 C CNN
 F 2 "" H 9450 1400 50  0000 C CNN
@@
 $EndComp
 $Comp
-L GND #PWR27
+L GND #PWR037
 U 1 1 56ECCB03
 P 9900 1400
-F 0 "#PWR27" H 9900 1150 50  0001 C CNN
+F 0 "#PWR037" H 9900 1150 50  0001 C CNN
 F 1 "GND" H 9900 1250 50  0000 C CNN
 F 2 "" H 9900 1400 50  0000 C CNN
@@
 $EndComp
 $Comp
-L GND #PWR29
+L GND #PWR038
 U 1 1 56ECCB7D
 P 10450 1400
-F 0 "#PWR29" H 10450 1150 50  0001 C CNN
+F 0 "#PWR038" H 10450 1150 50  0001 C CNN
 F 1 "GND" H 10450 1250 50  0000 C CNN
 F 2 "" H 10450 1400 50  0000 C CNN
@@
 $EndComp
 $Comp
-L GND #PWR24
+L GND #PWR039
 U 1 1 56ECD060
 P 9450 2200
-F 0 "#PWR24" H 9450 1950 50  0001 C CNN
+F 0 "#PWR039" H 9450 1950 50  0001 C CNN
 F 1 "GND" H 9450 2050 50  0000 C CNN
 F 2 "" H 9450 2200 50  0000 C CNN
@@
 $EndComp
 $Comp
-L GND #PWR28
+L GND #PWR040
 U 1 1 56ECD066
 P 9900 2200
-F 0 "#PWR28" H 9900 1950 50  0001 C CNN
+F 0 "#PWR040" H 9900 1950 50  0001 C CNN
 F 1 "GND" H 9900 2050 50  0000 C CNN
 F 2 "" H 9900 2200 50  0000 C CNN
@@
 $EndComp
 $Comp
-L GND #PWR30
+L GND #PWR041
 U 1 1 56ECD06C
 P 10450 2200
-F 0 "#PWR30" H 10450 1950 50  0001 C CNN
+F 0 "#PWR041" H 10450 1950 50  0001 C CNN
 F 1 "GND" H 10450 2050 50  0000 C CNN
 F 2 "" H 10450 2200 50  0000 C CNN
@@
 F 0 "C15" H 9910 1320 50  0000 L CNN
 F 1 "100nF" H 9910 1170 50  0000 L CNN
-F 2 "Capacitors_SMD:C_0402" H 9900 1250 50  0001 C CNN
+F 2 "Capacitors_SMD:C_0603" H 9900 1250 50  0001 C CNN
 F 3 "" H 9900 1250 50  0000 C CNN
 	1    9900 1250
@@
 F 0 "C17" H 10460 1320 50  0000 L CNN
 F 1 "100nF" H 10460 1170 50  0000 L CNN
-F 2 "Capacitors_SMD:C_0402" H 10450 1250 50  0001 C CNN
+F 2 "Capacitors_SMD:C_0603" H 10450 1250 50  0001 C CNN
 F 3 "" H 10450 1250 50  0000 C CNN
 	1    10450 1250
@@
 F 0 "C18" H 10460 2120 50  0000 L CNN
 F 1 "100nF" H 10460 1970 50  0000 L CNN
-F 2 "Capacitors_SMD:C_0402" H 10450 2050 50  0001 C CNN
+F 2 "Capacitors_SMD:C_0603" H 10450 2050 50  0001 C CNN
 F 3 "" H 10450 2050 50  0000 C CNN
 	1    10450 2050
@@
 F 0 "C16" H 9910 2120 50  0000 L CNN
 F 1 "100nF" H 9910 1970 50  0000 L CNN
-F 2 "Capacitors_SMD:C_0402" H 9900 2050 50  0001 C CNN
+F 2 "Capacitors_SMD:C_0603" H 9900 2050 50  0001 C CNN
 F 3 "" H 9900 2050 50  0000 C CNN
 	1    9900 2050
@@
 F 0 "C14" H 9460 2120 50  0000 L CNN
 F 1 "100nF" H 9460 1970 50  0000 L CNN
-F 2 "Capacitors_SMD:C_0402" H 9450 2050 50  0001 C CNN
+F 2 "Capacitors_SMD:C_0603" H 9450 2050 50  0001 C CNN
 F 3 "" H 9450 2050 50  0000 C CNN
 	1    9450 2050
@@
 $EndComp
 $Comp
-L GND #PWR25
+L GND #PWR042
 U 1 1 5792E9B8
 P 9450 3250
-F 0 "#PWR25" H 9450 3000 50  0001 C CNN
+F 0 "#PWR042" H 9450 3000 50  0001 C CNN
 F 1 "GND" H 9450 3100 50  0000 C CNN
 F 2 "" H 9450 3250 50  0000 C CNN
@@
 +9V
 $Comp
-L GND #PWR21
+L GND #PWR043
 U 1 1 56EAAE4F
 P 3700 2350
-F 0 "#PWR21" H 3700 2100 50  0001 C CNN
+F 0 "#PWR043" H 3700 2100 50  0001 C CNN
 F 1 "GND" H 3700 2200 50  0000 C CNN
 F 2 "" H 3700 2350 50  0000 C CNN
