File: hardware/Kicad_PCB_helios/DAC.sch (KiCad schematic (older format))
At the start: 4 parts, among them U5 DAC084S085C

Commit message: pull
Parts:
- added C33: 4.7uF, symbol C
- added C34, C35: 100nF, Capacitors_SMD:C_0603, symbol C
- added C36, C37: 10nF, Capacitors_SMD:C_0603, symbol C
- added C5: 4.7uF, Capacitors_SMD:CP_Elec_4x5.3, symbol C
- added U10, U11: DAC8531, TO_SOT_Packages_SMD:SOT-23-8_Handsoldering, symbol DAC8531
- C10, C12: footprint Capacitors_SMD:C_0402 -> Capacitors_SMD:C_0603
Connections:
- net 3.3V: now also C33.1, C34.1, C35.1, C5.1, U10.4 (VCC), U11.4 (VCC)
- net Din: now also U10.6 (DIN), U11.6 (DIN)
- net GND: now also C33.2, C34.2, C35.2, C36.2, C37.2, C5.2, U10.5 (GND), U11.5 (GND)
- net SCLK: now also U10.7 (SCLK), U11.7 (SCLK)
- net !SYNC renamed !SYNC-Quad
- new net !SYNC-X: U10.8 (~SYNC)
- new net !SYNC-Y: U11.8 (~SYNC)
- new net X: U10.1 (VOUT), U10.2 (VFB)
- new net X_SCALING: C36.1, U10.3 (VREF)
- new net Y: U11.1 (VOUT), U11.2 (VFB)
- new net Y_SCALING: C37.1, U11.3 (VREF)
