File: hardware/Kicad_PCB_helios/Helios.kicad_pcb (KiCad board)
At the start: 2 copper layers, 75.2 x 61.1 mm, 101 parts, among them P1 USB_B, P2 CONN_01X25-SHIELD, U1 IP4220CZ6, U2 AP2114, U3 AN431B, U4 ISA_DC-DC_converter, U5 DAC084S085C, U6 TL084_v, U7 LM358, U8 TL084_v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

Commit message: pull
Parts:
- removed ERASE: CONN_01X02, Connect:PINHEAD1-2
- removed P2: CONN_01X25-SHIELD, personal:DB25
- removed R33, R34: 1.65k, Resistors_SMD:R_0603
- removed REF** (x3): Fiducial_1mm_Dia_2.54mm_Outer_CopperTop, Fiducials:Fiducial_1mm_Dia_2.54mm_Outer_CopperTop
- added C34: 100nF, Capacitors_SMD:C_0603, F.Cu at (138.8, 145.8)
- added C35: 100nF, Capacitors_SMD:C_0603, F.Cu at (138.7, 150.2)
- added C36: 10nF, Capacitors_SMD:C_0603, F.Cu at (137.4, 144.8)
- added C37: 10nF, Capacitors_SMD:C_0603, F.Cu at (137.2, 149.4)
- added C5: 4.7uF, Capacitors_SMD:CP_Elec_4x5.3, F.Cu at (141.9, 153.5)
- added ERASE1: CONN_01X02, Pin_Headers:Pin_Header_Straight_1x02_Pitch2.54mm, F.Cu at (121.8, 128.9)
- added P3: CONN_02X13, Connectors:IDC_Header_Straight_26pins, F.Cu at (164.7, 115.0)
- added U10: DAC8531, TO_SOT_Packages_SMD:SOT-23-8_Handsoldering, F.Cu at (141.8, 144.1)
- added U11: DAC8531, TO_SOT_Packages_SMD:SOT-23-8_Handsoldering, F.Cu at (141.8, 148.2)
- added W1: TEST_1P, Connectors:1pin, F.Cu at (105.0, 156.0)
- added W2: TEST_1P, Connectors:1pin, F.Cu at (105.0, 105.0)
- added W3: TEST_1P, Connectors:1pin, F.Cu at (170.0, 156.0)
- added W4: TEST_1P, Connectors:1pin, F.Cu at (170.0, 105.0)
- added W5: TEST_1P, Symbols:WEEE-Logo_14x20mm_SilkScreen, B.Cu at (149.7, 129.9)
- C10, C12, C13, C14, C15, C16, C17, C18, C19, C2, C20, C21, C22, C25, C26, C27, C28, C3, C32, C7: footprint Capacitors_SMD:C_0402 -> Capacitors_SMD:C_0603
- C29, C31: footprint Capacitors_SMD:C_0402 -> Capacitors_SMD:C_0603_HandSoldering
- moved C2 2.83 mm to (110.2, 121.2)
- moved R11 2.13 mm to (161.9, 144.7)
- moved R35 2.13 mm to (147.3, 112.9)
- moved C10 1.97 mm to (146.7, 142.2)
- moved R3 1.90 mm to (162.1, 115.0)
- moved R4 1.90 mm to (162.1, 112.9)
- moved C28 1.60 mm to (120.9, 145.4), turned to 135 degrees
- moved C29 1.24 mm to (118.5, 143.1), turned to 315 degrees
- moved R39 1.08 mm to (157.1, 109.2)
- moved C31 1.05 mm to (115.8, 140.4), turned to 135 degrees
- moved C25 0.60 mm to (119.7, 139.5)
- moved C32 0.56 mm to (124.2, 145.9)
- moved C20 0.50 mm to (120.9, 135.7)
- moved C13 0.36 mm to (154.5, 145.4)
- moved R36 0.35 mm to (151.7, 119.7)
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Connections:
- net /Amplifiers/+9V renamed /+9V
- net /Amplifiers/+B renamed /+B
- net /Amplifiers/+G renamed /+G
- net /Amplifiers/+Intensity renamed /+Int
- net /Amplifiers/+R renamed /+R
- net /Amplifiers/+X renamed /+X
- net /Amplifiers/+Y renamed /+Y
- net /Amplifiers/-9V renamed /-9V
- net /Amplifiers/-X renamed /-X
- net /Amplifiers/-Y renamed /-Y
- net /Amplifiers/2.5V renamed /2.5V
- net /Amplifiers/B renamed /B
- net /Amplifiers/G renamed /G
- net /Amplifiers/Intensity renamed /Int
- net /Amplifiers/R renamed /R
- net /Amplifiers/Shutter renamed /Shutter
- net /Amplifiers/Shutter_Out renamed /Shutter_Out
- net /DAC/!SYNC renamed /DAC/!SYNC-Quad
- net /DAC/3.3V renamed /3.3V
- net /Power Regulation/5V renamed /VCC
- F1 pad 1: Net-(F1-Pad1) -> Net-(C2-Pad1)
- P1 pad 1: Net-(F1-Pad1) -> Net-(C2-Pad1)
- P1 pad 5: Net-(C2-Pad1) -> GND
- R10 pad 1: Net-(P2-Pad7) -> /X7
- R11 pad 1: Net-(P2-Pad13) -> /X13
- R3 pad 1: Net-(P2-Pad1) -> /X1
- R4 pad 1: Net-(P2-Pad14) -> /X14
- R5 pad 1: Net-(P2-Pad2) -> /X2
- R6 pad 1: Net-(P2-Pad15) -> /X15
- R7 pad 1: Net-(P2-Pad3) -> /X3
- R8 pad 1: Net-(P2-Pad5) -> /X5
- R9 pad 1: Net-(P2-Pad6) -> /X6
- U8 pad 10: Net-(R34-Pad1) -> /Amplifiers/Offset
- U8 pad 3: Net-(R33-Pad1) -> /Amplifiers/Offset
- U9 pad 29: (no net) -> /DAC/!SYNC-X
- U9 pad 30: (no net) -> /DAC/!SYNC-Y
- U9 pad 59: /Amplifiers/X -> /DAC/X_SCALING
- U9 pad 63: /Amplifiers/Y -> /DAC/Y_SCALING
Routing:
- net GND: track 138.7 -> 234.1 mm, vias 55 -> 53
- net /3.3V: track 95.3 -> 129.7 mm, vias 2 -> 5
- net /DAC/!SYNC-Y: track 0.00 -> 23.8 mm, vias 0 -> 2
- net /DAC/Y_SCALING: track 0.00 -> 21.9 mm
- net /DAC/X_SCALING: track 0.00 -> 20.9 mm
- net /Shutter_Out: track 45.7 -> 28.2 mm, vias 0 -> 2
- net Net-(F1-Pad1): track 17.2 -> 0.00 mm
- net /DAC/!SYNC-X: track 0.00 -> 16.7 mm, vias 0 -> 2
- net /DAC/Din: track 7.27 -> 23.7 mm
- net /Shutter: track 33.1 -> 45.6 mm
- net /Amplifiers/Offset: track 17.3 -> 29.7 mm, vias 0 -> 2
- net /DAC/SCLK: track 7.79 -> 18.2 mm
- net /2.5V: track 51.6 -> 41.6 mm
- net /Amplifiers/Y: track 45.6 -> 55.0 mm, vias 4 -> 5
- net Net-(P2-Pad15): track 7.49 -> 0.00 mm
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Other:
- board text added: "Helios Laser DAC Rev 2.0"
- board text removed: "Helios Laser DAC Rev 1.1"
