File: hardware/Kicad_PCB_helios/Helios.sch (KiCad schematic (older format))
At the start: 19 parts, among them P1 USB_B, P2 CONN_01X25-SHIELD, U1 IP4220CZ6

Commit message: pull
Parts:
- added J1: DB25, Connectors:DB25FD, symbol DB25
- added P3: CONN_02X13, Connectors:IDC_Header_Straight_26pins, symbol CONN_02X13
- added W1, W2, W3, W4: TEST_1P, Connectors:1pin, symbol TEST_1P
- C2, C3: footprint Capacitors_SMD:C_0402 -> Capacitors_SMD:C_0603
- P1: footprint Connect:USB_B -> (none)
- P2: footprint personal:DB25 -> (none)
Connections:
- net GND: now also P1.5 (shield), J1.0 (GND), J1.10, J1.11, J1.16 (P16), J1.18 (P18), J1.19 (P19), J1.20 (P20), J1.21 (P21), J1.22 (P22), J1.23 (P23), J1.24 (P24), J1.25 (P25), J1.8, J1.9, P3.10 (P10), P3.12 (P12), P3.14 (P14), P3.15 (P15), P3.16 (P16), P3.17 (P17), P3.18 (P18), P3.19 (P19), P3.20 (P20), P3.21 (P21), P3.22 (P22), P3.24 (P24), P3.26 (P26), P3.6 (P6), W1.1, W2.1, W3.1, W4.1
- net Interlock: now also J1.17 (P17), J1.4, P3.7 (P7), P3.8 (P8)
- net at F1.1, P1.1 (VBUS): now also C2.1
- net X1: now reaches P2.1 (P1), R3.1
- net X1: now also J1.1, P3.1 (P1)
- net X2: now reaches P2.2 (P2), R5.1
- net X2: now also J1.2, P3.3 (P3)
- net X3: now reaches P2.3 (P3), R7.1
- net X3: now also J1.3, P3.5 (P5)
- net X5: now reaches P2.5 (P5), R8.1
- net X5: now also J1.5, P3.9 (P9)
- net X6: now reaches P2.6 (P6), R9.1
- net X6: now also J1.6, P3.11 (P11)
- net X7: now reaches P2.7 (P7), R10.1
- net X7: now also J1.7, P3.13 (P13)
- net X13: now reaches P2.13 (P13), R11.1
- net X13: now also J1.13, P3.25 (P25)
- net X14: now reaches P2.14 (P14), R4.1
- net X14: now also J1.14 (P14), P3.2 (P2)
- net X15: now reaches P2.15 (P15), R6.1
- net X15: now also J1.15 (P15), P3.4 (P4)
Other:
- moved on the sheet: R10, R11, R3, R4, R5, R6, R7, R8, R9
