File: hardware/Kicad_PCB_helios/Helios.sch (KiCad schematic (older format))
At the start: 19 parts, among them P1 USB_B, P2 CONN_01X25-SHIELD, U1 IP4220CZ6

Commit message: fix some outdated schematics
Parts:
- P1: symbol USB_B -> USB_B-RESCUE-Helios
Changed lines of the file:
@@
 EESchema Schematic File Version 2
+LIBS:Helios-rescue
 LIBS:power
 LIBS:device
@@
 $EndSheet
 $Comp
-L USB_B P1
+L USB_B-RESCUE-Helios P1
 U 1 1 56B1FF91
 P 1150 2300
@@
 $EndSheet
 $Comp
-L GND #PWR6
+L GND #PWR01
 U 1 1 56B34131
 P 10750 4000
-F 0 "#PWR6" H 10750 3750 50  0001 C CNN
+F 0 "#PWR01" H 10750 3750 50  0001 C CNN
 F 1 "GND" H 10750 3850 50  0000 C CNN
 F 2 "" H 10750 4000 50  0000 C CNN
@@
 $EndComp
 $Comp
-L GND #PWR5
+L GND #PWR02
 U 1 1 56C4FEF7
 P 10700 2400
-F 0 "#PWR5" H 10700 2150 50  0001 C CNN
+F 0 "#PWR02" H 10700 2150 50  0001 C CNN
 F 1 "GND" H 10700 2250 50  0000 C CNN
 F 2 "" H 10700 2400 50  0000 C CNN
@@
 D+
 $Comp
-L GND #PWR2
+L GND #PWR03
 U 1 1 56ED04E3
 P 1450 2650
-F 0 "#PWR2" H 1450 2400 50  0001 C CNN
+F 0 "#PWR03" H 1450 2400 50  0001 C CNN
 F 1 "GND" H 1450 2500 50  0000 C CNN
 F 2 "" H 1450 2650 50  0000 C CNN
@@
 $EndComp
 $Comp
-L GND #PWR3
+L GND #PWR04
 U 1 1 5739A27B
 P 1850 3400
-F 0 "#PWR3" H 1850 3150 50  0001 C CNN
+F 0 "#PWR04" H 1850 3150 50  0001 C CNN
 F 1 "GND" H 1850 3250 50  0000 C CNN
 F 2 "" H 1850 3400 50  0000 C CNN
@@
 $EndComp
 $Comp
-L GND #PWR4
+L GND #PWR05
 U 1 1 575A19B8
 P 3600 3800
-F 0 "#PWR4" H 3600 3550 50  0001 C CNN
+F 0 "#PWR05" H 3600 3550 50  0001 C CNN
 F 1 "GND" H 3600 3650 50  0000 C CNN
 F 2 "" H 3600 3800 50  0000 C CNN
@@
 $EndComp
 $Comp
-L GND #PWR1
+L GND #PWR06
 U 1 1 575963D0
 P 1150 3450
-F 0 "#PWR1" H 1150 3200 50  0001 C CNN
+F 0 "#PWR06" H 1150 3200 50  0001 C CNN
 F 1 "GND" H 1150 3300 50  0000 C CNN
 F 2 "" H 1150 3450 50  0000 C CNN
