File: hardware/Kicad_PCB_helios/Power.sch (KiCad schematic (older format))
At the start: 11 parts, among them U2 AP2114, U3 AN431B, U4 ISA_DC-DC_converter

Commit message: pull
Parts:
- C7: footprint Capacitors_SMD:C_0402 -> Capacitors_SMD:C_0603
Changed lines of the file:
@@
 EESchema Schematic File Version 2
+LIBS:Helios-rescue
 LIBS:power
 LIBS:device
@@
 $EndComp
 $Comp
-L GND #PWR7
+L GND #PWR012
 U 1 1 56EC0DF6
 P 3100 6150
-F 0 "#PWR7" H 3100 5900 50  0001 C CNN
+F 0 "#PWR012" H 3100 5900 50  0001 C CNN
 F 1 "GND" H 3100 6000 50  0000 C CNN
 F 2 "" H 3100 6150 50  0000 C CNN
@@
 5V
 $Comp
-L GND #PWR9
+L GND #PWR013
 U 1 1 56ED02CC
 P 7500 3050
-F 0 "#PWR9" H 7500 2800 50  0001 C CNN
+F 0 "#PWR013" H 7500 2800 50  0001 C CNN
 F 1 "GND" H 7500 2900 50  0000 C CNN
 F 2 "" H 7500 3050 50  0000 C CNN
@@
 $EndComp
 $Comp
-L GND #PWR10
+L GND #PWR014
 U 1 1 56ED03CC
 P 8350 2500
-F 0 "#PWR10" H 8350 2250 50  0001 C CNN
+F 0 "#PWR014" H 8350 2250 50  0001 C CNN
 F 1 "GND" H 8350 2350 50  0000 C CNN
 F 2 "" H 8350 2500 50  0000 C CNN
@@
 -9V
 $Comp
-L GND #PWR12
+L GND #PWR015
 U 1 1 5703D8E0
 P 8550 2950
-F 0 "#PWR12" H 8550 2700 50  0001 C CNN
+F 0 "#PWR015" H 8550 2700 50  0001 C CNN
 F 1 "GND" H 8550 2800 50  0000 C CNN
 F 2 "" H 8550 2950 50  0000 C CNN
@@
 $EndComp
 $Comp
-L GND #PWR11
+L GND #PWR016
 U 1 1 5703D96C
 P 8550 2050
-F 0 "#PWR11" H 8550 1800 50  0001 C CNN
+F 0 "#PWR016" H 8550 1800 50  0001 C CNN
 F 1 "GND" H 8550 1900 50  0000 C CNN
 F 2 "" H 8550 2050 50  0000 C CNN
@@
 $EndComp
 $Comp
-L GND #PWR8
+L GND #PWR017
 U 1 1 573CF740
 P 3350 3050
-F 0 "#PWR8" H 3350 2800 50  0001 C CNN
+F 0 "#PWR017" H 3350 2800 50  0001 C CNN
 F 1 "GND" H 3350 2900 50  0000 C CNN
 F 2 "" H 3350 3050 50  0000 C CNN
@@
 Shunt reference is UNSTABLE when bypassed with 10^3 to 10^6 pF so 100nF can't be used alone
 $Comp
-L PWR_FLAG #FLG1
+L PWR_FLAG #FLG018
 U 1 1 575B50A4
 P 1950 2200
-F 0 "#FLG1" H 1950 2295 50  0001 C CNN
+F 0 "#FLG018" H 1950 2295 50  0001 C CNN
 F 1 "PWR_FLAG" H 1950 2380 50  0000 C CNN
 F 2 "" H 1950 2200 50  0000 C CNN
@@
 	8250 2600 8650 2600
 Wire Wire Line
-	8250 2500 8350 2500
-Wire Wire Line
 	8550 2350 8550 2400
 Connection ~ 8550 2400
@@
 F 0 "C7" H 6675 2800 50  0000 L CNN
 F 1 "100nF" H 6675 2600 50  0000 L CNN
-F 2 "Capacitors_SMD:C_0402" H 6688 2550 50  0001 C CNN
+F 2 "Capacitors_SMD:C_0603" H 6688 2550 50  0001 C CNN
 F 3 "" H 6650 2700 50  0000 C CNN
 	1    6650 2700
@@
 Connection ~ 6650 3000
 $Comp
-L PWR_FLAG #FLG2
+L PWR_FLAG #FLG019
 U 1 1 5792E8E7
 P 6750 2400
-F 0 "#FLG2" H 6750 2495 50  0001 C CNN
+F 0 "#FLG019" H 6750 2495 50  0001 C CNN
 F 1 "PWR_FLAG" H 6750 2580 50  0000 C CNN
 F 2 "" H 6750 2400 50  0000 C CNN
@@
 Wire Wire Line
 	1950 2950 3350 2950
+Wire Wire Line
+	8250 2500 8350 2500
 $EndSCHEMATC
